Commit message: Updated turtlebot3_burger_with_ns.gazebo.xacro, turtlebot3_burger_with_ns.urdf.xacro: based on the namespace updates on gazebo, robot_state_publisher, gazebo_ros::spawn_model, etc.

File: turtlebot3_description/urdf/turtlebot3_burger_with_ns.gazebo.xacro (robot description, xacro)
@@ -1,10 +1,10 @@
 <?xml version="1.0"?>
 <robot name="turtlebot3_burger_sim" xmlns:xacro="http://ros.org/wiki/xacro">
-  <xacro:arg name="laser_visual" default="true"/>
+  <xacro:arg name="laser_visual" default="false"/>
   <xacro:arg name="imu_visual"   default="false"/>
-  <gazebo reference="$(arg ns)/base_link">
+  <gazebo reference="base_link">
     <material>Gazebo/DarkGrey</material>
   </gazebo>
-  <gazebo reference="$(arg ns)/wheel_left_link">
+  <gazebo reference="wheel_left_link">
     <mu1>0.1</mu1>
     <mu2>0.1</mu2>
@@ -16,5 +16,5 @@
     <material>Gazebo/FlatBlack</material>
   </gazebo>
-  <gazebo reference="$(arg ns)/wheel_right_link">
+  <gazebo reference="wheel_right_link">
     <mu1>0.1</mu1>
     <mu2>0.1</mu2>
@@ -26,5 +26,5 @@
     <material>Gazebo/FlatBlack</material>
   </gazebo>
-  <gazebo reference="$(arg ns)/caster_back_link">
+  <gazebo reference="caster_back_link">
     <mu1>0.1</mu1>
     <mu2>0.1</mu2>
@@ -35,5 +35,5 @@
     <material>Gazebo/FlatBlack</material>
   </gazebo>
-  <gazebo reference="$(arg ns)/imu_link">
+  <gazebo reference="imu_link">
     <sensor type="imu" name="imu">
       <always_on>true</always_on>
@@ -44,6 +44,6 @@
   <gazebo>
     <plugin name="turtlebot3_burger_controller" filename="libgazebo_ros_diff_drive.so">
-      <commandTopic>$(arg ns)/cmd_vel</commandTopic>
-      <odometryTopic>$(arg ns)/odom</odometryTopic>
+      <commandTopic>cmd_vel</commandTopic>
+      <odometryTopic>odom</odometryTopic>
       <odometryFrame>$(arg ns)/odom</odometryFrame>
       <odometrySource>world</odometrySource>
@@ -55,6 +55,6 @@
       <legacyMode>false</legacyMode>
       <updateRate>30</updateRate>
-      <leftJoint>$(arg ns)/wheel_left_joint</leftJoint>
-      <rightJoint>$(arg ns)/wheel_right_joint</rightJoint>
+      <leftJoint>wheel_left_joint</leftJoint>
+      <rightJoint>wheel_right_joint</rightJoint>
       <wheelSeparation>0.160</wheelSeparation>
       <wheelDiameter>0.066</wheelDiameter>
@@ -67,8 +67,8 @@
     <plugin name="imu_plugin" filename="libgazebo_ros_imu.so">
       <alwaysOn>true</alwaysOn>
-      <bodyName>$(arg ns)/imu_link</bodyName>
-      <frameName>$(arg ns)/imu_link</frameName>
-      <topicName>$(arg ns)/imu</topicName>
-      <serviceName>$(arg ns)/imu_service</serviceName>
+      <bodyName>imu_link</bodyName>
+      <frameName>imu_link</frameName>
+      <topicName>imu</topicName>
+      <serviceName>imu_service</serviceName>
       <gaussianNoise>0.0</gaussianNoise>
       <updateRate>0</updateRate>
@@ -92,24 +92,22 @@
     </plugin>
   </gazebo>
-  <gazebo reference="$(arg ns)/base_scan">
+  <gazebo reference="base_scan">
     <material>Gazebo/FlatBlack</material>
-    <sensor type="gpu_ray" name="lds_lfcd_sensor">
+    <sensor type="ray" name="lds_lfcd_sensor">
       <pose>0 0 0 0 0 0</pose>
       <visualize>$(arg laser_visual)</visualize>
-      <update_rate>50</update_rate>
+      <update_rate>5</update_rate>
       <ray>
         <scan>
           <horizontal>
-            <samples>512</samples>
+            <samples>360</samples>
             <resolution>1</resolution>
-            <min_angle>-2.356</min_angle>
-            <!--max_angle>6.28319</max_angle-->
-            <max_angle>2.356</max_angle>
+            <min_angle>0.0</min_angle>
+            <max_angle>6.28319</max_angle>
           </horizontal>
         </scan>
         <range>
-          <!--min>0.12</min-->
-          <min>0.1</min>
-          <max>4.0</max>
+          <min>0.120</min>
+          <max>3.5</max>
           <resolution>0.015</resolution>
         </range>
@@ -120,6 +118,6 @@
         </noise>
       </ray>
-      <plugin name="gazebo_ros_lds_lfcd_controller" filename="libgazebo_ros_gpu_laser.so">
-        <topicName>$(arg ns)/scan</topicName>
+      <plugin name="gazebo_ros_lds_lfcd_controller" filename="libgazebo_ros_laser.so">
+        <topicName>scan</topicName>
         <frameName>$(arg ns)/base_scan</frameName>
       </plugin>

File: turtlebot3_description/urdf/turtlebot3_burger_with_ns.urdf.xacro (robot description, xacro)
@@ -4,11 +4,11 @@
   <xacro:include filename="$(find turtlebot3_description)/urdf/common_properties.xacro"/>
   <xacro:include filename="$(find turtlebot3_description)/urdf/turtlebot3_burger_with_ns.gazebo.xacro"/>
-  <link name="$(arg ns)/base_footprint"/>
-  <joint name="$(arg ns)/base_joint" type="fixed">
-    <parent link="$(arg ns)/base_footprint"/>
-    <child link="$(arg ns)/base_link"/>
+  <link name="base_footprint"/>
+  <joint name="base_joint" type="fixed">
+    <parent link="base_footprint"/>
+    <child link="base_link"/>
     <origin xyz="0.0 0.0 0.010" rpy="0 0 0"/>
   </joint>
-  <link name="$(arg ns)/base_link">
+  <link name="base_link">
     <visual>
       <origin xyz="-0.032 0 0.0" rpy="0 0 0"/>
@@ -32,11 +32,11 @@
     </inertial>
   </link>
-  <joint name="$(arg ns)/wheel_left_joint" type="continuous">
-    <parent link="$(arg ns)/base_link"/>
-    <child link="$(arg ns)/wheel_left_link"/>
+  <joint name="wheel_left_joint" type="continuous">
+    <parent link="base_link"/>
+    <child link="wheel_left_link"/>
     <origin xyz="0.0 0.08 0.023" rpy="-1.57 0 0"/>
     <axis xyz="0 0 1"/>
   </joint>
-  <link name="$(arg ns)/wheel_left_link">
+  <link name="wheel_left_link">
     <visual>
       <origin xyz="0 0 0" rpy="1.57 0 0"/>
@@ -60,11 +60,11 @@
       </inertial>
   </link>
-  <joint name="$(arg ns)/wheel_right_joint" type="continuous">
-    <parent link="$(arg ns)/base_link"/>
-    <child link="$(arg ns)/wheel_right_link"/>
+  <joint name="wheel_right_joint" type="continuous">
+    <parent link="base_link"/>
+    <child link="wheel_right_link"/>
     <origin xyz="0.0 -0.080 0.023" rpy="-1.57 0 0"/>
     <axis xyz="0 0 1"/>
   </joint>
-  <link name="$(arg ns)/wheel_right_link">
+  <link name="wheel_right_link">
     <visual>
       <origin xyz="0 0 0" rpy="1.57 0 0"/>
@@ -88,10 +88,10 @@
       </inertial>
   </link>
-  <joint name="$(arg ns)/caster_back_joint" type="fixed">
-    <parent link="$(arg ns)/base_link"/>
-    <child link="$(arg ns)/caster_back_link"/>
+  <joint name="caster_back_joint" type="fixed">
+    <parent link="base_link"/>
+    <child link="caster_back_link"/>
     <origin xyz="-0.081 0 -0.004" rpy="-1.57 0 0"/>
   </joint>
-  <link name="$(arg ns)/caster_back_link">
+  <link name="caster_back_link">
     <collision>
       <origin xyz="0 0.001 0" rpy="0 0 0"/>
@@ -108,16 +108,16 @@
     </inertial>
   </link>
-  <joint name="$(arg ns)/imu_joint" type="fixed">
-    <parent link="$(arg ns)/base_link"/>
-    <child link="$(arg ns)/imu_link"/>
+  <joint name="imu_joint" type="fixed">
+    <parent link="base_link"/>
+    <child link="imu_link"/>
     <origin xyz="-0.032 0 0.068" rpy="0 0 0"/>
   </joint>
-  <link name="$(arg ns)/imu_link"/>
-  <joint name="$(arg ns)/scan_joint" type="fixed">
-    <parent link="$(arg ns)/base_link"/>
-    <child link="$(arg ns)/base_scan"/>
+  <link name="imu_link"/>
+  <joint name="scan_joint" type="fixed">
+    <parent link="base_link"/>
+    <child link="base_scan"/>
     <origin xyz="-0.032 0 0.172" rpy="0 0 0"/>
   </joint>
-  <link name="$(arg ns)/base_scan">
+  <link name="base_scan">
     <visual>
       <origin xyz="0 0 0.0" rpy="0 0 0"/>
